Commit message: Corrected 2nd Lidar position

File: robots/youbot_base_only_navigation.urdf.xacro (robot description, xacro)
@@ -16,5 +16,5 @@
   <!-- sensors -->
   <xacro:include filename="$(find youbot_description)/urdf/sensors/hokuyo_urg04_laser.urdf.xacro"/>
-   	<xacro:include filename="$(find youbot_description)/urdf/sensors/hokuyo_urg04_laser2.urdf.xacro"/>
+  <xacro:include filename="$(find youbot_description)/urdf/sensors/hokuyo_urg04_laser2.urdf.xacro"/>
   <!-- Now we can start using the macros xacro:included above to define the actual youbot -->
   <!-- The first use of a macro.  This one was defined in base.urdf.xacro above.

File: urdf/sensors/hokuyo_urg04_laser2.urdf.xacro (robot description, xacro)
@@ -8,5 +8,5 @@
     <joint name="${name}_hokuyo_urg04_laser_joint" type="fixed">
       <axis xyz="0 1 0" />
-      <insert_block name="origin" />
+      <xacro:insert_block name="origin" />
       <parent link="${parent}_link"/>
       <child link="${name}_link"/>
@@ -20,8 +20,7 @@
       <visual>
       	<origin xyz="0 0 0" rpy="0 0 0" />
-	<geometry>
-		<mesh filename="package://youbot_description/meshes/sensors/hokuyo.dae" />
-	</geometry>
-	<material name="DarkGrey" />
+        <geometry>
+            <mesh filename="package://youbot_description/meshes/sensors/hokuyo.dae" />
+        </geometry>
       </visual>
       <collision>
